File: haptic-linear-slider.kicad_pcb (KiCad board)
At the start: 2 copper layers, 130.5 x 33.8 mm, 56 parts, among them IC1 DIO54335TST6, IC2 TLV61048DBVR, J1 SWD_TagConnect, J2 USB_C_Receptacle_USB2.0_16P, J3 TBC05-02-1-G-G, SW1 SW_Push, SW2 SW_Push, U1 RP2354_60QFN, U2 PSM01-081A-103B2, U3 DRV8876PWPR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

Commit message: 3D models are mostly working
Parts:
- C11, C12, C13: footprint Capacitor_SMD:C_0402_1005Metric -> _Footprints:C_0402_1005Metric_small_pads
- C32: footprint MyFootprints:CAPPRD350W52D800H1300 -> _Footprints:CAPPRD350W52D800H1300
- D1: footprint MyFootprints:SODFL3618X110N -> _Footprints:SODFL3618X110N
- IC1: footprint MyFootprints:SOT95P280X90-6N -> _Footprints:SOT95P280X90-6N
- IC2: footprint MyFootprints:SOT95P280X145-6N -> _Footprints:SOT95P280X145-6N
- J3: footprint MyFootprints:TBC05021GG -> _Footprints:TBC05021GG
- L1: value AMRM00101040100MA1 (10u) -> 10u; footprint MyFootprints:AMRM00101040100MA1 -> _Footprints:AMRM00101040100MA1
- L2: value MPL-SE6040-6R8 (6u8) -> 6u8; footprint MyFootprints:MPLSE60406R8 -> _Footprints:MPLSE60406R8
- U2: footprint MyFootprints:PSM01081A103B2 -> _Footprints:PSM01081A103B2
- U3: footprint MyFootprints:SOP65P640X120-17N -> _Footprints:SOP65P640X120-17N
- Y1: footprint Crystal:Crystal_SMD_3225-4Pin_3.2x2.5mm -> _Footprints:Crystal_SMD_HC49-US
- moved Y1 6.42 mm to (323.9, 222.4)
Connections:
- J2 pad SH: (no net) -> GND
