File: haptic-linear-slider.kicad_sch (KiCad schematic)
At the start: 76 parts, among them IC1 DIO54335TST6, IC2 TLV61048DBVR, J1 SWD_TagConnect, J2 USB_C_Receptacle_USB2.0_16P, J3 TBC05-02-1-G-G, SW1 SW_Push, SW2 SW_Push, U1 RP2354_60QFN, U2 PSM01-081A-103B2, U3 DRV8876PWPR, Y1 ABM8-272-T3

Commit message: Test
Other:
- note added: "Come mai questo GND non è collegato a nulla?"
Changed lines of the file:
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@@
+		)
+	)
+	(text "Come mai questo GND non è collegato a nulla?\n"
+		(exclude_from_sim no)
+		(at 64.516 190.754 0)
+		(effects
+			(font
+				(size 1.27 1.27)
+			)
+			(justify left bottom)
 		)
 	)

Commit message: Test
Parts:
- C1, C2, C3, C7, C8, C9: footprint 0 -> Capacitor_SMD:C_1210_3225Metric_Pad1.33x2.70mm_HandSolder; Manufacturer_Name (none) -> Samsung Electro-Mechanics; Manufacturer_Part_Number (none) -> CL32B106KBJNNWE; Mouser Part Number (none) -> 187-CL32B106KBJNNWE; Mouser Price/Stock (none) -> https://www.mouser.it/en/ProductDetail/Samsung-Electro-Mech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
Other:
- note added: "Bisogna capire che condensatori comprare per C4 e C5 Ho visto che però è già stato assiciato un footprint"
- note added: "Gengis, le NetTie vanno tolte secondo Chat GPT"

Commit message: Condensatori
Parts:
- C10: Manufacturer_Name (none) -> Samsung Electro-Mechanics; Manufacturer_Part_Number (none) -> CL21B105KBFNNNG; Mouser Part Number (none) -> 187-CL21B105KBFNNNG; Mouser Price/Stock (none) -> https://www.mouser.it/en/ProductDetail/Samsung-Electro-Mech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
- C11, C12, C13: Manufacturer_Name (none) -> Samsung Electro-Mechanics; Manufacturer_Part_Number (none) -> CL05A475MO5NUNC; Mouser Part Number (none) -> 187-CL05A475MO5NUNC; Mouser Price/Stock (none) -> https://www.mouser.it/en/ProductDetail/Samsung-Electro-Mech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
- C27, C28, C29, C30, C6: Manufacturer_Name (none) -> Samsung Electro-Mechanics; Manufacturer_Part_Number (none) -> CL21B104KBFNNNG; Mouser Part Number (none) -> 187-CL21B104KBFNNNG; Mouser Price/Stock (none) -> Capacitor_SMD:C_0603_1608Metric_Pad1.08x0.95mm_HandSolder
- C4, C5: Manufacturer_Name (none) -> Samsung Electro-Mechanics; Manufacturer_Part_Number (none) -> CL10C150JB8NNN; Mouser Part Number (none) -> 187-CL10C150JB8NNNC; Mouser Price/Stock (none) -> https://www.mouser.it/en/ProductDetail/Samsung-Electro-Mech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
Other:
- note removed: "Come mai questo GND non è collegato a nulla?"

Commit message: Condensatori
Parts:
- C14, C16, C17, C18, C19, C20, C21, C22, C23, C24, C25, C26: footprint Capacitor_SMD:C_0603_1608Metric_Pad1.08x0.95mm_HandSolder -> _Footprints:C_0402_1005Metric_small_pads; Manufacturer_Name (none) -> Samsung Electro-Mechanics; Manufacturer_Part_Number (none) -> CL05B104KO5NFNC; Mouser Part Number (none) -> 187-CL05B104KO5NFNC; Mouser Price/Stock (none) -> https://www.mouser.it/en/ProductDetail/Samsung-Electro-Mech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
- C15: value 4u7 -> 100n; footprint Capacitor_SMD:C_0603_1608Metric_Pad1.08x0.95mm_HandSolder -> _Footprints:C_0402_1005Metric_small_pads; Manufacturer_Name (none) -> Samsung Electro-Mechanics; Manufacturer_Part_Number (none) -> CL05B104KO5NFNC; Mouser Part Number (none) -> 187-CL05B104KO5NFNC; Mouser Price/Stock (none) -> https://www.mouser.it/en/ProductDetail/Samsung-Electro-Mech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
- C31: Manufacturer_Name (none) -> Samsung Electro-Mechanics; Manufacturer_Part_Number (none) -> CL05B223KB5NNNC; Mouser Part Number (none) -> 187-CL05B223KB5NNNC; Mouser Price/Stock (none) -> https://www.mouser.it/en/ProductDetail/Samsung-Electro-Mech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
